Commit message: Add end effector plate

File: urdf/deflector.xacro (robot description, xacro)
@@ -79,5 +79,5 @@
     <dynamics damping="10.0"/>
   </joint>
-  <!-- Gantry -->
+  <!-- Gantry Cart -->
   <link name="link3">
     <collision>
@@ -130,4 +130,34 @@
     </inertial>
   </link>
+<!-- End Effector -->
+<xacro:if value="$(arg end_effector_plate)">
+    <joint name="end_effector_joint" type="fixed">
+      <!-- link origin with respect to the origin of the body of the parent link -->
+      <origin xyz="0 ${y_width_l4/2} ${y_width_l4/2}" rpy="${pi/2} 0 0" /> <!-- Placed at the center of one end of the parent link (link 4) -->
+      <parent link="link4"/>
+      <child link="end_effector_plate"/>
+    </joint>
+ <!-- End Effector Link -->
+  <link name="end_effector_plate">
+    <collision>
+    <xacro:insert_block name="ee_plate_link_origin" />
+      <geometry>
+	   <box size="${x_width_ee_plate} ${y_width_ee_plate} ${height_ee_plate}"/>
+      </geometry>
+    </collision>
+    <visual>
+      <xacro:insert_block name="ee_plate_link_origin" />
+      <geometry>
+	   <box size="${x_width_ee_plate} ${y_width_ee_plate} ${height_ee_plate}"/>
+      </geometry>
+    </visual>
+    <inertial>
+      <xacro:insert_block name="ee_plate_link_origin" />
+      <mass value="${mass_ee_plate}"/>
+      <xacro:inertial_cuboid mass="${mass_ee_plate}" x_width="${x_width_ee_plate}" y_width="${y_width_ee_plate}" length="${height_ee_plate}" >
+      </xacro:inertial_cuboid>
+    </inertial>
+  </link>
+</xacro:if>
 <!-- declare transmissions and actuators required to interface with ROS control -->
 <!-- defines ressource of hardware_interface::EffortJointInterface -->

File: urdf/properties.xacro (robot description, xacro)
@@ -7,4 +7,5 @@
 <xacro:property name="mass_gantry" value="0.1" />
 <xacro:property name="mass_l4" value="10.0" />
+<xacro:property name="mass_ee_plate" value="1.0" />
 <xacro:property name="axel_offset" value="0.1" />
 <!-- Size of Robot Axes -->
@@ -21,4 +22,7 @@
 <xacro:property name="y_width_l4" value="0.2" />
 <xacro:property name="lenght_l4" value="1.0" />
+<xacro:property name="x_width_ee_plate" value="0.3" /> <!-- parallel to axis of lenght of link 2 -->
+<xacro:property name="y_width_ee_plate" value="0.6" /> <!-- parallel to axis of lenght of link 1 -->
+<xacro:property name="height_ee_plate" value="0.05" />
 <!-- Origin Positions and Orientations -->
 <!-- Set the origin pose on the base link (as child frame) -->
@@ -38,3 +42,9 @@
   <origin xyz="0 ${-lenght_l4/2+y_width_gantry/2} ${y_width_l4/2}" rpy="${pi/2} 0 0" />
 </xacro:property>
+<!-- Set the origin pose on the end effector link (child frame = end_effector) -->
+<xacro:property name="ee_plate_link_origin">
+  <origin xyz="0.0  0.0 ${-height_ee_plate/2}" rpy="0 0 0" /> <!-- Place at the surface of the plate -->
+</xacro:property>
+<!-- End Effector Configuration -->
+<xacro:arg name="end_effector_plate" default="true"/>
 </robot>
